Commit message: add camera

File: urdf/diffdam.xacro (robot description, xacro)
@@ -149,3 +149,48 @@
     </sensor>
   </gazebo>
+   <joint name="camera_joint" type="fixed">
+    <origin xyz="0.000 0.000 0.15" rpy="0 0 0"/>
+    <parent link="link_chassis"/>
+    <child link="camera_frame"/>
+  </joint>
+  <link name="camera_frame"/>
+   <gazebo reference="camera_frame">
+    <sensor type="camera" name="camera1">
+      <update_rate>30.0</update_rate>
+      <camera name="head">
+        <horizontal_fov>1.3962634</horizontal_fov>
+        <image>
+          <width>800</width>
+          <height>800</height>
+          <format>R8G8B8</format>
+        </image>
+        <clip>
+          <near>0.02</near>
+          <far>300</far>
+        </clip>
+        <noise>
+          <type>gaussian</type>
+          <!-- Noise is sampled independently per pixel on each frame.
+               That pixel's noise value is added to each of its color
+               channels, which at that point lie in the range [0,1]. -->
+          <mean>0.0</mean>
+          <stddev>0.007</stddev>
+        </noise>
+      </camera>
+      <plugin name="camera_controller" filename="libgazebo_ros_camera.so">
+        <alwaysOn>true</alwaysOn>
+        <updateRate>0.0</updateRate>
+        <cameraName>diffdam/camera1</cameraName>
+        <imageTopicName>image_raw</imageTopicName>
+        <cameraInfoTopicName>camera_info</cameraInfoTopicName>
+        <frameName>camera_link</frameName>
+        <hackBaseline>0.07</hackBaseline>
+        <distortionK1>0.0</distortionK1>
+        <distortionK2>0.0</distortionK2>
+        <distortionK3>0.0</distortionK3>
+        <distortionT1>0.0</distortionT1>
+        <distortionT2>0.0</distortionT2>
+      </plugin>
+    </sensor>
+  </gazebo>
 </robot>

Commit message: edit max range lidar

File: urdf/diffdam.xacro (robot description, xacro)
@@ -134,5 +134,5 @@
         <range>
           <min>0.10</min>
-          <max>10.0</max>
+          <max>15.0</max>
           <resolution>0.01</resolution>
         </range>
@@ -150,22 +150,22 @@
   </gazebo>
    <joint name="camera_joint" type="fixed">
-    <origin xyz="0.000 0.000 0.15" rpy="0 0 0"/>
+    <origin xyz="0.000 0.000 0.2" rpy="0 -1.570796 0"/>
     <parent link="link_chassis"/>
-    <child link="camera_frame"/>
+    <child link="camera_link"/>
   </joint>
-  <link name="camera_frame"/>
-   <gazebo reference="camera_frame">
+  <link name="camera_link"/>
+   <gazebo reference="camera_link">
     <sensor type="camera" name="camera1">
-      <update_rate>30.0</update_rate>
-      <camera name="head">
-        <horizontal_fov>1.3962634</horizontal_fov>
+      <update_rate>60.0</update_rate>
+      <camera name="fiducial_cam">
+        <!-- <horizontal_fov>1.3962634</horizontal_fov> -->
         <image>
-          <width>800</width>
-          <height>800</height>
+          <width>1080</width>
+          <height>720</height>
           <format>R8G8B8</format>
         </image>
         <clip>
           <near>0.02</near>
-          <far>300</far>
+          <far>3500</far>
         </clip>
         <noise>
